File: hardware/pcb/adapter-heltec_v3/Heltec v3 adapter.kicad_pcb (KiCad board)
At the start: 2 copper layers, 53.6 x 58.4 mm, 2 parts, among them U1 ESP32_LORA_V2.0

Commit message: Initial boards for raw prototyping
Parts:
- added C1: C_Polarized, Capacitor_THT:CP_Radial_D8.0mm_P3.50mm, F.Cu at (132.8, 75.2)
- added C2: C, Capacitor_THT:C_Rect_L4.0mm_W2.5mm_P2.50mm, F.Cu at (140.2, 75.2)
- added J1: Conn_01x02_Pin, Connector_PinHeader_2.54mm:PinHeader_1x02_P2.54mm_Vertical, F.Cu at (140.2, 79.0)
Connections:
- U1 pad J2_3: VDD -> VEXT
- U1 pad J2_4: VDD -> VEXT
- U2 pad 1: unconnected-(U2-GND_A-Pad1) -> GND
- U2 pad 12: VDD -> unconnected-(U2-VBAT_C-Pad12)
- U2 pad 16: unconnected-(U2-GND_D-Pad16) -> GND
- U2 pad 2: unconnected-(U2-VBAT_A-Pad2) -> VDD
- U2 pad 22: (no net) -> GND
- U2 pad 23: (no net) -> GND
- U2 pad 24: (no net) -> GND
- U2 pad 25: (no net) -> GND
- U2 pad 6: unconnected-(U2-GND_B-Pad6) -> GND
Routing:
- net IO5: track 0.00 -> 39.8 mm
- net IO6: track 0.00 -> 39.6 mm
- net IO7: track 0.00 -> 39.3 mm
- net VDD: track 0.00 -> 29.9 mm
- net IO4: track 0.00 -> 27.5 mm
- net IO2: track 0.00 -> 13.6 mm
- net IO1: track 0.00 -> 13.6 mm
- net IO3: track 0.00 -> 13.4 mm
- net GND: track 0.00 -> 3.83 mm
- net 3V3: track 0.00 -> 2.54 mm
- net VEXT: track 0.00 -> 2.54 mm
- added copper zone on B.Cu, net GND
Other:
- board text added: "Heltec V3 adapter v1.0 TwinOak Standard Repeater"
