File: hardware/pcb/platform-board/platform-board.kicad_sch (KiCad schematic)
At the start: 9 parts, among them J1 Conn_01x09_Pin, J2 Conn_01x05_Pin, J3 Conn_01x05_Pin, J4 Conn_01x05_Pin, J5 Conn_01x05_Pin

Commit message: Initial boards for raw prototyping
Parts:
- J1: footprint Connector_PinHeader_2.54mm:PinHeader_1x09_P2.54mm_Horizontal -> TwinOak platform footprints:82155700
Changed lines of the file:
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@@
 		)
 		(instances
-			(project "standard-repeater-design-v2"
+			(project "platform-board"
 				(path "/06a38798-314b-43d0-92f7-26c13b6d6633"
 					(reference "#PWR03")
@@
 		)
 		(instances
-			(project "standard-repeater-design-v2"
+			(project "platform-board"
 				(path "/06a38798-314b-43d0-92f7-26c13b6d6633"
 					(reference "H3")
@@
 		)
 		(instances
-			(project "standard-repeater-design-v2"
+			(project "platform-board"
 				(path "/06a38798-314b-43d0-92f7-26c13b6d6633"
 					(reference "#PWR06")
@@
 			)
 		)
-		(property "Footprint" "Connector_PinHeader_2.54mm:PinHeader_1x09_P2.54mm_Horizontal"
+		(property "Footprint" "TwinOak platform footprints:82155700"
 			(at 109.22 91.44 0)
 			(hide yes)
@@
 		)
 		(instances
-			(project "standard-repeater-design-v2"
+			(project "platform-board"
 				(path "/06a38798-314b-43d0-92f7-26c13b6d6633"
 					(reference "J1")
@@
 		)
 		(instances
-			(project "standard-repeater-design-v2"
+			(project "platform-board"
 				(path "/06a38798-314b-43d0-92f7-26c13b6d6633"
 					(reference "#PWR09")
@@
 		)
 		(instances
-			(project "standard-repeater-design-v2"
+			(project "platform-board"
 				(path "/06a38798-314b-43d0-92f7-26c13b6d6633"
 					(reference "#PWR01")
@@
 		)
 		(instances
-			(project "standard-repeater-design-v2"
+			(project "platform-board"
 				(path "/06a38798-314b-43d0-92f7-26c13b6d6633"
 					(reference "#PWR07")
@@
 		)
 		(instances
-			(project "standard-repeater-design-v2"
+			(project "platform-board"
 				(path "/06a38798-314b-43d0-92f7-26c13b6d6633"
 					(reference "H1")
@@
 		)
 		(instances
-			(project "standard-repeater-design-v2"
+			(project "platform-board"
 				(path "/06a38798-314b-43d0-92f7-26c13b6d6633"
 					(reference "J2")
@@
 		)
 		(instances
-			(project "standard-repeater-design-v2"
+			(project "platform-board"
 				(path "/06a38798-314b-43d0-92f7-26c13b6d6633"
 					(reference "H4")
@@
 		)
 		(instances
-			(project "standard-repeater-design-v2"
+			(project "platform-board"
 				(path "/06a38798-314b-43d0-92f7-26c13b6d6633"
 					(reference "J3")
@@
 		)
 		(instances
-			(project "standard-repeater-design-v2"
+			(project "platform-board"
 				(path "/06a38798-314b-43d0-92f7-26c13b6d6633"
 					(reference "#PWR02")
@@
 		)
 		(instances
-			(project "standard-repeater-design-v2"
+			(project "platform-board"
 				(path "/06a38798-314b-43d0-92f7-26c13b6d6633"
 					(reference "#PWR05")
@@
 		)
 		(instances
-			(project "standard-repeater-design-v2"
+			(project "platform-board"
 				(path "/06a38798-314b-43d0-92f7-26c13b6d6633"
 					(reference "J5")
@@
 		)
 		(instances
-			(project "standard-repeater-design-v2"
+			(project "platform-board"
 				(path "/06a38798-314b-43d0-92f7-26c13b6d6633"
 					(reference "J4")
@@
 		)
 		(instances
-			(project "standard-repeater-design-v2"
+			(project "platform-board"
 				(path "/06a38798-314b-43d0-92f7-26c13b6d6633"
 					(reference "#PWR08")
@@
 		)
 		(instances
-			(project "standard-repeater-design-v2"
+			(project "platform-board"
 				(path "/06a38798-314b-43d0-92f7-26c13b6d6633"
 					(reference "H2")
@@
 		)
 		(instances
-			(project "standard-repeater-design-v2"
+			(project "platform-board"
 				(path "/06a38798-314b-43d0-92f7-26c13b6d6633"
 					(reference "#PWR04")

Commit message: Cleanup
Parts:
- J1: footprint TwinOak platform footprints:82155700 -> TwinOak:82155700

Commit message: Platform rewire
Connections:
- net at J2.2 (Pin_2), J3.2 (Pin_2): now also J1.3 (Pin_3); no longer J1.2 (Pin_2)
- net at J2.3 (Pin_3), J3.3 (Pin_3): now also J1.5 (Pin_5); no longer J1.3 (Pin_3)
- net at J2.4 (Pin_4), J3.4 (Pin_4): now also J1.7 (Pin_7); no longer J1.4 (Pin_4)
- net at J2.5 (Pin_5), J3.5 (Pin_5): now also J1.9 (Pin_9); no longer J1.5 (Pin_5)
- net at J4.2 (Pin_2), J5.2 (Pin_2): now also J1.2 (Pin_2); no longer J1.6 (Pin_6)
- net at J4.3 (Pin_3), J5.3 (Pin_3): now also J1.4 (Pin_4); no longer J1.7 (Pin_7)
- net at J4.4 (Pin_4), J5.4 (Pin_4): now also J1.6 (Pin_6); no longer J1.8 (Pin_8)
- net at J4.5 (Pin_5), J5.5 (Pin_5): now also J1.8 (Pin_8); no longer J1.9 (Pin_9)
Other:
- note added: "J1 wired for flat ribbon fan-out at the D-sub solder cups: ribbon conductor -> cup order 1,6,2,7,3,8,4,9,5 (conductor 10 unused). Red stripe (conductor 1) at the D-sub pin-1 end. Do NOT wire 1:1 by pin number. Same map as a standard IDC DE-9. See INTERCONNECT.md."
Changed lines of the file:
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@@
-	(wire
-		(pts
-			(xy 114.3 93.98)
-			(xy 135.89 93.98)
-		)
-		(stroke
-			(width 0)
-			(type default)
-		)
-	)
 	(wire
 		(pts
@@
 	(wire
 		(pts
-			(xy 114.3 96.52)
-			(xy 134.62 96.52)
-		)
-		(stroke
-			(width 0)
-			(type default)
-		)
-	)
-	(wire
-		(pts
-			(xy 114.3 88.9)
-			(xy 133.35 88.9)
-		)
-		(stroke
-			(width 0)
-			(type default)
-		)
-	)
-	(wire
-		(pts
 			(xy 119.38 81.28)
 			(xy 119.38 76.2)
@@
 	(wire
 		(pts
-			(xy 114.3 99.06)
-			(xy 133.35 99.06)
-		)
-		(stroke
-			(width 0)
-			(type default)
-		)
-	)
-	(wire
-		(pts
 			(xy 170.18 96.52)
 			(xy 134.62 96.52)
@@
 	(wire
 		(pts
-			(xy 114.3 91.44)
-			(xy 132.08 91.44)
-		)
-		(stroke
-			(width 0)
-			(type default)
-		)
-	)
-	(wire
-		(pts
 			(xy 135.89 83.82)
 			(xy 135.89 71.12)
@@
 	(wire
 		(pts
-			(xy 114.3 86.36)
-			(xy 134.62 86.36)
-		)
-		(stroke
-			(width 0)
-			(type default)
-		)
-	)
-	(wire
-		(pts
-			(xy 114.3 101.6)
-			(xy 132.08 101.6)
-		)
-		(stroke
-			(width 0)
-			(type default)
-		)
-	)
-	(wire
-		(pts
 			(xy 171.45 93.98)
 			(xy 135.89 93.98)
-		)
-		(stroke
-			(width 0)
-			(type default)
-		)
-	)
-	(wire
-		(pts
-			(xy 114.3 83.82)
-			(xy 135.89 83.82)
 		)
 		(stroke
@@
 		)
 	)
+	(wire
+		(pts
+			(xy 114.3 83.82)
+			(xy 120.65 83.82)
+		)
+		(stroke
+			(width 0)
+			(type default)
+		)
+	)
+	(wire
+		(pts
+			(xy 120.65 83.82)
+			(xy 120.65 93.98)
+		)
+		(stroke
+			(width 0)
+			(type default)
+		)
+	)
+	(wire
+		(pts
+			(xy 120.65 93.98)
+			(xy 135.89 93.98)
+		)
+		(stroke
+			(width 0)
+			(type default)
+		)
+	)
+	(wire
+		(pts
+			(xy 114.3 86.36)
+			(xy 121.92 86.36)
+		)
+		(stroke
+			(width 0)
+			(type default)
+		)
+	)
+	(wire
+		(pts
+			(xy 121.92 86.36)
+			(xy 121.92 83.82)
+		)
+		(stroke
+			(width 0)
+			(type default)
+		)
+	)
+	(wire
+		(pts
+			(xy 121.92 83.82)
+			(xy 135.89 83.82)
+		)
+		(stroke
+			(width 0)
+			(type default)
+		)
+	)
+	(wire
+		(pts
+			(xy 114.3 88.9)
+			(xy 127 88.9)
+		)
+		(stroke
+			(width 0)
+			(type default)
+		)
+	)
+	(wire
+		(pts
+			(xy 127 88.9)
+			(xy 127 96.52)
+		)
+		(stroke
+			(width 0)
+			(type default)
+		)
+	)
+	(wire
+		(pts
+			(xy 127 96.52)
+			(xy 134.62 96.52)
+		)
+		(stroke
+			(width 0)
+			(type default)
+		)
+	)
+	(wire
+		(pts
+			(xy 114.3 91.44)
+			(xy 123.19 91.44)
+		)
+		(stroke
+			(width 0)
+			(type default)
+		)
+	)
+	(wire
+		(pts
+			(xy 123.19 91.44)
+			(xy 123.19 86.36)
+		)
+		(stroke
+			(width 0)
+			(type default)
+		)
+	)
+	(wire
+		(pts
+			(xy 123.19 86.36)
+			(xy 134.62 86.36)
+		)
+		(stroke
+			(width 0)
+			(type default)
+		)
+	)
+	(wire
+		(pts
+			(xy 114.3 93.98)
+			(xy 118.11 93.98)
+		)
+		(stroke
+			(width 0)
+			(type default)
+		)
+	)
+	(wire
+		(pts
+			(xy 118.11 93.98)
+			(xy 118.11 99.06)
+		)
+		(stroke
+			(width 0)
+			(type default)
+		)
+	)
+	(wire
+		(pts
+			(xy 118.11 99.06)
+			(xy 133.35 99.06)
+		)
+		(stroke
+			(width 0)
+			(type default)
+		)
+	)
+	(wire
+		(pts
+			(xy 114.3 96.52)
+			(xy 125.73 96.52)
+		)
+		(stroke
+			(width 0)
+			(type default)
+		)
+	)
+	(wire
+		(pts
+			(xy 125.73 96.52)
+			(xy 125.73 95.25)
+		)
+		(stroke
+			(width 0)
+			(type default)
+		)
+	)
+	(wire
+		(pts
+			(xy 125.73 95.25)
+			(xy 128.27 95.25)
+		)
+		(stroke
+			(width 0)
+			(type default)
+		)
+	)
+	(wire
+		(pts
+			(xy 128.27 95.25)
+			(xy 128.27 88.9)
+		)
+		(stroke
+			(width 0)
+			(type default)
+		)
+	)
+	(wire
+		(pts
+			(xy 128.27 88.9)
+			(xy 133.35 88.9)
+		)
+		(stroke
+			(width 0)
+			(type default)
+		)
+	)
+	(wire
+		(pts
+			(xy 114.3 99.06)
+			(xy 116.84 99.06)
+		)
+		(stroke
+			(width 0)
+			(type default)
+		)
+	)
+	(wire
+		(pts
+			(xy 116.84 99.06)
+			(xy 116.84 101.6)
+		)
+		(stroke
+			(width 0)
+			(type default)
+		)
+	)
+	(wire
+		(pts
+			(xy 116.84 101.6)
+			(xy 132.08 101.6)
+		)
+		(stroke
+			(width 0)
+			(type default)
+		)
+	)
+	(wire
+		(pts
+			(xy 114.3 101.6)
+			(xy 115.57 101.6)
+		)
+		(stroke
+			(width 0)
+			(type default)
+		)
+	)
+	(wire
+		(pts
+			(xy 115.57 101.6)
+			(xy 115.57 92.71)
+		)
+		(stroke
+			(width 0)
+			(type default)
+		)
+	)
+	(wire
+		(pts
+			(xy 115.57 92.71)
+			(xy 124.46 92.71)
+		)
+		(stroke
+			(width 0)
+			(type default)
+		)
+	)
+	(wire
+		(pts
+			(xy 124.46 92.71)
+			(xy 124.46 91.44)
+		)
+		(stroke
+			(width 0)
+			(type default)
+		)
+	)
+	(wire
+		(pts
+			(xy 124.46 91.44)
+			(xy 132.08 91.44)
+		)
+		(stroke
+			(width 0)
+			(type default)
+		)
+	)
+	(text "J1 wired for flat ribbon fan-out at the D-sub solder cups:\nribbon conductor -> cup order 1,6,2,7,3,8,4,9,5 (conductor 10 unused).\nRed stripe (conductor 1) at the D-sub pin-1 end. Do NOT wire 1:1 by pin\nnumber. Same map as a standard IDC DE-9. See INTERCONNECT.md."
+		(exclude_from_sim no)
+		(at 99.06 111.76 0)
+		(effects
+			(font
+				(size 1.27 1.27)
+			)
+			(justify left bottom)
+		)
+	)

Commit message: Last pre-production updates
Parts:
- J1, J2, J3, J4, J5: now left out of the parts list
Changed lines of the file:
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@@
 		(body_style 1)
 		(exclude_from_sim no)
-		(in_bom yes)
-		(on_board yes)
-		(in_pos_files yes)
+		(in_bom no)
+		(on_board yes)
+		(in_pos_files no)
 		(dnp no)
 		(fields_autoplaced yes)
@@
 		(body_style 1)
 		(exclude_from_sim no)
-		(in_bom yes)
-		(on_board yes)
-		(in_pos_files yes)
+		(in_bom no)
+		(on_board yes)
+		(in_pos_files no)
 		(dnp no)
 		(fields_autoplaced yes)
@@
 		(body_style 1)
 		(exclude_from_sim no)
-		(in_bom yes)
-		(on_board yes)
-		(in_pos_files yes)
+		(in_bom no)
+		(on_board yes)
+		(in_pos_files no)
 		(dnp no)
 		(fields_autoplaced yes)
@@
 		(body_style 1)
 		(exclude_from_sim no)
-		(in_bom yes)
-		(on_board yes)
-		(in_pos_files yes)
+		(in_bom no)
+		(on_board yes)
+		(in_pos_files no)
 		(dnp no)
 		(fields_autoplaced yes)
@@
 		(body_style 1)
 		(exclude_from_sim no)
-		(in_bom yes)
-		(on_board yes)
-		(in_pos_files yes)
-		(dnp no)
-		(fields_autoplaced yes)
+		(in_bom no)
+		(on_board yes)
+		(in_pos_files no)
+		(dnp no)
+		(fields_autoplaced yes)
