File: hardware/pcb/connector-board-a/connector-board-a.kicad_sch (KiCad schematic)
At the start: 26 parts, among them J1 DE9_Pins, J2 8-215570-0, J3 J_ENV, Q3 2N7002, U4 TPS63001, U5 BME280

Commit message: Parts ordered!
Parts:
- J3: now left out of the parts list
Changed lines of the file:
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@@
 		(body_style 1)
 		(exclude_from_sim no)
-		(in_bom yes)
+		(in_bom no)
 		(on_board yes)
-		(in_pos_files yes)
+		(in_pos_files no)
 		(dnp no)
 		(property "Reference" "J3"
